File: pcb/display_power.kicad_sch (KiCad schematic)
At the start: 44 parts, among them Q1 MMBTA06, Q2 Q_PNP_BCEC, Q7 MMBTA06, U5 PAM2804AAB010, U6 SC189ZSKTRT, U7 LMR51430, U8 FODM217A

Commit message: Saved pcb
Parts:
- R15, R36: value 33k -> 3k3
- R33: value 33k -> 10k
Changed lines of the file:
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@@
 			)
 		)
-		(property "Value" "33k"
+		(property "Value" "3k3"
 			(at 157.48 69.8499 0)
 			(effects
@@
 			)
 		)
-		(property "Value" "33k"
+		(property "Value" "10k"
 			(at 186.6899 46.99 0)
 			(effects
@@
 			)
 		)
-		(property "Value" "33k"
+		(property "Value" "3k3"
 			(at 157.48 57.1499 0)
 			(effects
